File: tests/fixtures/benchmark/qfp_fanout.kicad_pcb (KiCad board)
At the start: 2 copper layers, 46 x 46 mm, 17 parts, among them J1 GPIO-A, J2 GPIO-B, U1 MCU, Y1 8MHz

Commit message: fix(bench): qfp_fanout ran its headers off the board, and the router was scored on it
The violations clustered at y = 45.5 to 46.1 on a board 46mm tall, which
is what gave it away. Two 21-pin headers are 50.8mm of pins: three pads
per header sat past the outline. The fixture has been like that since it
landed two commits later than it should have been checked, and its
ratchet has been in CI guarding a board nobody could make.

A 46mm edge holds fifteen pins at 2.54mm once margins are taken, so two
sides cannot hold forty-eight. kicad_emit.header grew an `along_x`
option and the headers are one per edge. Checked rather than eyeballed -
every pad against the outline:

  pads outside the board outline: 0 []

Regenerating shift_driver through the shared emitter leaves it
byte-identical, so the change is confined to the board that needed it.

The valid board is much harder, which is the honest outcome. Escaping to
four edges rather than two:

  before  1177 routes, 343 after, 331 introduced, 183 shorts
  after   1971 routes, 676 after, 665 introduced, 424 shorts

Its band was re-measured with it: 606 to 665 across prices 0.22..0.28,
59 violations wide, narrower than the 102 the broken board showed. The
ratchet is the new value plus that band, 735 / 500, and
benchmark_all_fixtures_drc passes on it.

  cargo fmt --check                                       clean
  cargo clippy --workspace --all-targets -- -D warnings   clean
  cargo test --workspace --exclude cypcb-desktop          no failures
Parts:
- added J3: GPIO, Connector_PinHeader_2.54mm:PinHeader_1x12_P2.54mm_Vertical, F.Cu at (109.0, 63.0)
- added J4: GPIO, Connector_PinHeader_2.54mm:PinHeader_1x12_P2.54mm_Vertical, F.Cu at (109.0, 103.0)
- J1: value GPIO-A -> GPIO; footprint Connector_PinHeader_2.54mm:PinHeader_1x20_P2.54mm_Vertical -> Connector_PinHeader_2.54mm:PinHeader_1x12_P2.54mm_Vertical
- J2: value GPIO-B -> GPIO; footprint Connector_PinHeader_2.54mm:PinHeader_1x20_P2.54mm_Vertical -> Connector_PinHeader_2.54mm:PinHeader_1x12_P2.54mm_Vertical
- moved J1 6.03 mm to (103.0, 69.0)
- moved J2 6.03 mm to (143.0, 69.0)
Connections:
- J1 pad 12: IO11 -> VCC
- J2 pad 1: IO22 -> IO11
- J2 pad 10: IO31 -> IO20
- J2 pad 11: IO32 -> IO21
- J2 pad 12: IO33 -> GND
- J2 pad 2: IO23 -> IO12
- J2 pad 3: IO24 -> IO13
- J2 pad 4: IO25 -> IO14
- J2 pad 5: IO26 -> IO15
- J2 pad 6: IO27 -> IO16
- J2 pad 7: IO28 -> IO17
- J2 pad 8: IO29 -> IO18
- J2 pad 9: IO30 -> IO19

Commit message: test(bench): ask every fixture whether it is a board, and find an importer defect
Nothing had ever asked the obvious question of a benchmark fixture: is
this a board somebody could make? Asking it turned up more than expected.

The importer keys its footprint library by library name alone -
`if !library.contains(&library_key)` in pcb_parser.rs - so two parts
sharing a name and differing in geometry collapse into whichever was read
first. qfp_fanout's file puts two of its four headers along x; the model
had all four along y, so two of them ran off the board in the model while
the file was correct. Any KiCad board carrying a rotated or modified
variant of a footprint imports wrong.

The measurement was wrong twice before it was worth believing. The first
version squared each pad - max(width, height) on both axes, the bound the
routing grid uses - and reported eleven of qfp_fanout's pads as off the
board where a check against their real extents found none; an LQFP pad is
1.5 by 0.3mm. The second was an awk that matched the library string twice
per footprint and read the wrong block. Neither reached a claim, because
each contradicted an earlier measurement and the contradiction was chased
rather than explained away.

The fixture works around the defect by giving the horizontal pair a
library name of their own, and is now clean: 0 pads outside the outline.
That moved the board a third time, so it was measured a third time:

  1504 routes, 336 after, 336 introduced, 179 shorts
  band 296 to 336 across prices 0.22..0.28, 40 violations wide
  ratchet 376 / 260

every_fixture_is_a_board_somebody_could_make.rs counts off-board pads per
fixture and holds each against what is known:

  stm32_breakout   8 pads   two ten-pin headers past its 65mm height
  multi_ic        10 pads   an inductor and a transformer 50mm to the left
  shift_driver     6 pads   bypass capacitors 3mm above the top edge

A new fixture with copper off the board fails; these three are named with
their count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
Parts:
- J3, J4: footprint Connector_PinHeader_2.54mm:PinHeader_1x12_P2.54mm_Vertical -> Connector_PinHeader_2.54mm:PinHeader_1x12_P2.54mm_Horizontal
Changed lines of the file:
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@@
     (pad "12" thru_hole oval (at 0.0 27.94) (size 1.7 1.7) (drill 1.0) (layers "*.Cu" "*.Mask") (net 2 "GND"))
   )
-  (footprint "Connector_PinHeader_2.54mm:PinHeader_1x12_P2.54mm_Vertical"
+  (footprint "Connector_PinHeader_2.54mm:PinHeader_1x12_P2.54mm_Horizontal"
     (layer "F.Cu")
     (at 109.030 63.000)
     (property "Reference" "J3")
     (property "Value" "GPIO")
-    (property "Footprint" "Connector_PinHeader_2.54mm:PinHeader_1x12_P2.54mm_Vertical")
+    (property "Footprint" "Connector_PinHeader_2.54mm:PinHeader_1x12_P2.54mm_Horizontal")
     (pad "1" thru_hole rect (at 0.0 0.0) (size 1.7 1.7) (drill 1.0) (layers "*.Cu" "*.Mask") (net 29 "IO22"))
     (pad "2" thru_hole oval (at 2.54 0.0) (size 1.7 1.7) (drill 1.0) (layers "*.Cu" "*.Mask") (net 30 "IO23"))
@@
     (pad "12" thru_hole oval (at 27.94 0.0) (size 1.7 1.7) (drill 1.0) (layers "*.Cu" "*.Mask") (net 1 "VCC"))
   )
-  (footprint "Connector_PinHeader_2.54mm:PinHeader_1x12_P2.54mm_Vertical"
+  (footprint "Connector_PinHeader_2.54mm:PinHeader_1x12_P2.54mm_Horizontal"
     (layer "F.Cu")
     (at 109.030 103.000)
     (property "Reference" "J4")
     (property "Value" "GPIO")
-    (property "Footprint" "Connector_PinHeader_2.54mm:PinHeader_1x12_P2.54mm_Vertical")
+    (property "Footprint" "Connector_PinHeader_2.54mm:PinHeader_1x12_P2.54mm_Horizontal")
     (pad "1" thru_hole rect (at 0.0 0.0) (size 1.7 1.7) (drill 1.0) (layers "*.Cu" "*.Mask") (net 40 "IO33"))
     (pad "2" thru_hole oval (at 2.54 0.0) (size 1.7 1.7) (drill 1.0) (layers "*.Cu" "*.Mask") (net 41 "IO34"))
