File: tests/fixtures/benchmark/shift_driver.kicad_pcb (KiCad board)
At the start: 2 copper layers, 68 x 48 mm, 55 parts, among them J1 Ctrl, U1 74HC595, U2 74HC595, U3 74HC595

Commit message: fix(benchmark): the last two fixtures with copper off the board
stm32_breakout carried 8 pads outside its own outline and shift_driver 6.
Both were recorded in KNOWN_OFF_BOARD and reported to the owner as a blocked
decision for a dozen fires.

It was never an owner decision. Every reason it was blocked on - that
repairing a fixture moves its ratchet and the tables drawn from it - is work
done four times since without asking, on qfp_fanout, multi_ic and
plane_board. The blocker was stale and kept being repeated.

stm32_breakout had two ten-pin headers at y = 90. Ten pins at 2.54mm is
22.86mm, so the last four ran up to 7.9mm past a top edge at 105. They moved
to y = 80.

shift_driver had three bypass capacitors at y = -3.4, above the board
entirely, placed there to clear a DIP courtyard. The DIP starts at y = 4.0 and
reaches about 2.9 with its courtyard, so they moved to y = 1.5 - inside the
board and clear of it. Fixed at the generator, so make_shift_driver.py and the
board it writes agree.

Making them fabricable improved the routing sharply, which is the argument for
doing it at all:

  board            routes        violations      shorts
  stm32_breakout   908 -> 899    239 -> 180      136 -> 93
  shift_driver     700 -> 671    81 -> 65        33 -> 34

Pads off the board had been forcing the router into the edge region.

  led_blink: 21 routes, 2 violations against 2, 0 shorts against 0
  stm32_breakout: 899 routes, 180 against 210, 93 shorts against 136
  multi_ic: 945 routes, 291 against 354, 187 shorts against 210
  shift_driver: 671 routes, 65 against 77, 34 shorts against 40
  qfp_fanout: 1478 routes, 309 against 376, 147 shorts against 260
  plane_board: 181 routes, 28 against 37, 13 shorts against 18

Violation ratchets tighten to measured plus each board's measured band: 239 ->
210 and 93 -> 77. The shorts ratchets stay where they were rather than being
tightened by a number nobody measured, since neither board has a measured
shorts band. They are loose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
Parts:
- moved C1 4.90 mm to (115.8, 61.5)
- moved C2 4.90 mm to (133.8, 61.5)
- moved C3 4.90 mm to (151.8, 61.5)
Changed lines of the file:
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@@
   (footprint "Resistor_SMD:R_0805_2012Metric"
     (layer "F.Cu")
-    (at 115.800 56.600)
+    (at 115.800 61.500)
     (property "Reference" "C1")
     (property "Value" "100nF")
@@
   (footprint "Resistor_SMD:R_0805_2012Metric"
     (layer "F.Cu")
-    (at 133.800 56.600)
+    (at 133.800 61.500)
     (property "Reference" "C2")
     (property "Value" "100nF")
@@
   (footprint "Resistor_SMD:R_0805_2012Metric"
     (layer "F.Cu")
-    (at 151.800 56.600)
+    (at 151.800 61.500)
     (property "Reference" "C3")
     (property "Value" "100nF")
