File: tests/fixtures/benchmark/stm32_breakout.kicad_pcb (KiCad board)
At the start: 2 copper layers, 75 x 65 mm, 29 parts, among them J1 USB_C, J2 SWD, J3 GPIO_L, J4 GPIO_R, SW1 RESET, U1 STM32F103C8T6, U2 AMS1117-3.3, U3 USBLC6-2SC6, Y1 8MHz

Commit message: fix(benchmark): the copper the fixtures shipped was lines between part centres
multi_ic reported 32 pieces of copper touching copper at 0.00mm before
anything was routed. Reading the segments settled what they were:

  (segment (start 65 45) (end 90 62) ...)
  (segment (start 90 62) (end 100 70) ...)
  (segment (start 100 70) (end 110 62) ...)

65,45 is U4's origin, 90,62 is C1's, 100,70 is U1's. These are straight lines
drawn between part centres, so they cross every package on the way and short
against the pads they pass. All three fixtures that carried copper carried the
same decoration, shorting 1, 13 and 32 times respectively.

Removed: 3 segments and 2 vias from led_blink, 8 and 4 from stm32_breakout, 15
and 10 from multi_ic. All three now ship zero shorts.

led_blink keeps copper and it is real copper: one trace from R1 pad 2 at
(120.48, 65) to D1 pad 1 at (124.25, 65), both on LED_ANODE, adjacent parts,
nothing in between. The import path still has a fixture to prove itself on
rather than losing the coverage along with the decoration.

Every ratchet is unchanged, which is the proof this fed no measurement:

  led_blink: 21 routes, 2 violations against 2, 0 shorts against 0
  stm32_breakout: 908 routes, 239 against 239, 136 shorts against 136
  multi_ic: 945 routes, 291 against 354, 187 shorts against 210
  shift_driver: 700 routes, 81 against 93, 33 shorts against 40
  qfp_fanout: 1478 routes, 309 against 376, 147 shorts against 260
  plane_board: 181 routes, 28 against 37, 13 shorts against 18

The benchmark routes from scratch and never read it. What did read it was
cypcb check, the viewer, and the CLI's board loader - everything a person
actually points at a board.

Three test files leaned on it and were repointed rather than deleted. The
parse expectations say 1 segment and 0 vias for led_blink and no copper for
the other two, and the origin test - which exists to catch copper imported
without subtracting the board corner - measures against the new trace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
Routing:
- net VCC_3V3: track 28.8 -> 0.00 mm, vias 2 -> 0
- net NRST: track 14.1 -> 0.00 mm
- net USB_DP: track 9.43 -> 0.00 mm
- net LED2_K: track 5.00 -> 0.00 mm
- net LED1_K: track 5.00 -> 0.00 mm
- net I2C_SDA: track 5.00 -> 0.00 mm
- net GND: track 3.00 -> 0.00 mm, vias 2 -> 0
Changed lines of the file:
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@@
   )
   ; -- Reference traces --
-  (segment (start 92 55) (end 108 65) (width 0.25) (layer "F.Cu") (net 1))
-  (segment (start 108 65) (end 115 72) (width 0.25) (layer "F.Cu") (net 1))
-  (segment (start 85 72) (end 90 80) (width 0.25) (layer "F.Cu") (net 4))
-  (segment (start 130 60) (end 135 60) (width 0.2) (layer "F.Cu") (net 29))
-  (segment (start 130 64) (end 135 64) (width 0.2) (layer "F.Cu") (net 30))
-  (segment (start 115 72) (end 125 82) (width 0.2) (layer "F.Cu") (net 6))
-  (segment (start 125 85) (end 125 88) (width 0.2) (layer "F.Cu") (net 2))
-  (segment (start 140 82) (end 145 82) (width 0.2) (layer "F.Cu") (net 33))
-  (via (at 100 72) (size 0.8) (drill 0.4) (layers "F.Cu" "B.Cu") (net 2))
-  (via (at 120 72) (size 0.8) (drill 0.4) (layers "F.Cu" "B.Cu") (net 2))
-  (via (at 130 72) (size 0.8) (drill 0.4) (layers "F.Cu" "B.Cu") (net 1))
-  (via (at 95 65) (size 0.8) (drill 0.4) (layers "F.Cu" "B.Cu") (net 1))
 )

Commit message: fix(benchmark): the last two fixtures with copper off the board
stm32_breakout carried 8 pads outside its own outline and shift_driver 6.
Both were recorded in KNOWN_OFF_BOARD and reported to the owner as a blocked
decision for a dozen fires.

It was never an owner decision. Every reason it was blocked on - that
repairing a fixture moves its ratchet and the tables drawn from it - is work
done four times since without asking, on qfp_fanout, multi_ic and
plane_board. The blocker was stale and kept being repeated.

stm32_breakout had two ten-pin headers at y = 90. Ten pins at 2.54mm is
22.86mm, so the last four ran up to 7.9mm past a top edge at 105. They moved
to y = 80.

shift_driver had three bypass capacitors at y = -3.4, above the board
entirely, placed there to clear a DIP courtyard. The DIP starts at y = 4.0 and
reaches about 2.9 with its courtyard, so they moved to y = 1.5 - inside the
board and clear of it. Fixed at the generator, so make_shift_driver.py and the
board it writes agree.

Making them fabricable improved the routing sharply, which is the argument for
doing it at all:

  board            routes        violations      shorts
  stm32_breakout   908 -> 899    239 -> 180      136 -> 93
  shift_driver     700 -> 671    81 -> 65        33 -> 34

Pads off the board had been forcing the router into the edge region.

  led_blink: 21 routes, 2 violations against 2, 0 shorts against 0
  stm32_breakout: 899 routes, 180 against 210, 93 shorts against 136
  multi_ic: 945 routes, 291 against 354, 187 shorts against 210
  shift_driver: 671 routes, 65 against 77, 34 shorts against 40
  qfp_fanout: 1478 routes, 309 against 376, 147 shorts against 260
  plane_board: 181 routes, 28 against 37, 13 shorts against 18

Violation ratchets tighten to measured plus each board's measured band: 239 ->
210 and 93 -> 77. The shorts ratchets stay where they were rather than being
tightened by a number nobody measured, since neither board has a measured
shorts band. They are loose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
Parts:
- moved J3 10.0 mm to (85.0, 80.0)
- moved J4 10.0 mm to (145.0, 80.0)
Changed lines of the file:
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@@
   (footprint "Connector_PinHeader_2.54mm:PinHeader_1x10_P2.54mm_Vertical"
     (layer "F.Cu")
-    (at 85 90)
+    (at 85 80)
     (property "Reference" "J3")
     (property "Value" "GPIO_L")
@@
   (footprint "Connector_PinHeader_2.54mm:PinHeader_1x10_P2.54mm_Vertical"
     (layer "F.Cu")
-    (at 145 90)
+    (at 145 80)
     (property "Reference" "J4")
     (property "Value" "GPIO_R")
